File: plates/mx/lumberjack-full.kicad_pcb (KiCad board)
At the start: 2 copper layers, 285.8 x 95.3 mm, 0 parts

Commit message: Add copper outline to MX plates
Routing:
- net (no net): vias 1 -> 0
Other:
- outline, holes or cut-outs redrawn

Commit message: Fix copper outline missing on the back side of MX split plates
Changed lines of the file:
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@@
       (drillshape 0)
       (scaleselection 1)
-      (outputdirectory "gerbers")
+      (outputdirectory "../gerbers")
     )
   )
   (net 0 "")
-  (gr_rect (start 161.806617 133.945875) (end 273.8449 40.719546) (layer "F.Cu") (width 0.2) (fill solid))
-  (gr_rect (start -9.52504 133.945875) (end 102.513243 40.719546) (layer "F.Cu") (width 0.2) (fill solid))
   (gr_rect (start 162.64009 79.772178) (end 177.88009 95.012178) (layer "F.Mask") (width 0.1) (fill solid))
   (gr_rect (start 67.389722 79.77221) (end 82.629722 95.01221) (layer "F.Mask") (width 0.1) (fill solid))
@@
     (style (thickness 0.15) (arrow_length 1.27) (text_position_mode 0) (extension_height 0.58642) (extension_offset 0) keep_text_aligned)
   )
-  (zone (net 0) (net_name "") (layer "F.Cu") (hatch edge 0.508)
+  (zone (net 0) (net_name "") (layers F&B.Cu) (hatch edge 0.508)
+    (connect_pads (clearance 0))
+    (min_thickness 0.254) (filled_areas_thickness no)
+    (fill yes (thermal_gap 0.508) (thermal_bridge_width 0.508))
+    (polygon
+      (pts
+        (xy 102.399984 133.799978)
+        (xy -9.498746 133.801366)
+        (xy -9.398734 41.001366)
+        (xy 102.399996 40.999978)
+      )
+    )
+  )
+  (zone (net 0) (net_name "") (layers F&B.Cu) (hatch edge 0.508)
     (connect_pads (clearance 0.508))
     (min_thickness 0.254) (filled_areas_thickness no)
@@
     )
   )
-  (zone (net 0) (net_name "") (layer "B.Cu") (hatch edge 0.508)
-    (connect_pads (clearance 0.508))
+  (zone (net 0) (net_name "") (layers F&B.Cu) (hatch edge 0.508)
+    (connect_pads (clearance 0))
     (min_thickness 0.254) (filled_areas_thickness no)
     (fill yes (thermal_gap 0.508) (thermal_bridge_width 0.508))
     (polygon
       (pts
-        (xy 275 135)
-        (xy -10.8 135)
-        (xy -10.7 39.7)
-        (xy 275 39.7)
+        (xy 273.799934 133.799313)
+        (xy 161.901204 133.800701)
+        (xy 162.001216 41.000701)
+        (xy 273.799946 40.999313)
       )
     )
